File: zepto_receiver_elrs.sch (KiCad schematic (older format))
At the start: 54 parts, among them J1 u.fl, SW1 SW_Push, U1 STM32WLE5JBI6, U2 NCP160, U3 BGS12PL6E6327XTSA1, Y1 32MHz

Commit message: updated layout, adjusted courtyards, updated schematic pdf
Parts:
- C1, C13, C14, C15, C16, C17, C18, C19, C2, C20, C21, C22, C23, C24, C25, C26, C4, C6, C8: footprint Capacitor_SMD:C_0201_0603Metric -> ftprnts:C_0201_0603Metric_dense
- C10, C7: footprint ftprnts:0805_low_esl_cap_avx_w_via -> ftprnts:0805_low_esl_cap_avx_w_via_dense
- C11, C9: footprint ftprnts:0805_low_esl_cap_avx -> ftprnts:0805_low_esl_cap_avx_w_via_dense
- C3, C5: footprint Capacitor_SMD:C_0402_1005Metric -> ftprnts:L_0402_1005Metric_dense
- L2, L3, L4, L5, L6: footprint Inductor_SMD:L_0402_1005Metric -> ftprnts:L_0402_1005Metric_dense
- R1, R2, R3, R4, R5: footprint Resistor_SMD:R_0201_0603Metric -> ftprnts:R_0201_0603Metric_dense
Other:
- note added: "Only 50mV drouput -\n supply with 3,3V is possible"
- note removed: "Oonly 50mV drouput -\n supply with 3,3V is possible"
