File: zepto_receiver_elrs_20210313_1419.kicad_pcb (KiCad board)
At the start: 4 copper layers, 9.5 x 7.5 mm, 43 parts, among them J1 u.fl, SW1 SW_Push, U1 STM32WLE5JBI6, U2 NCP160, U3 BGS12PL6E6327XTSA1, U4 0900FM15D0039, U5 ECS-TXO-25CSMV-320-AM-TR

Commit message: adjust schematic, further layout work
Parts:
- removed C4: 1µF, ftprnts:C_0201_0603Metric_dense
- removed C7: 2.2uF, ftprnts:0805_low_esl_cap_avx
- removed C9: 2.2uF, ftprnts:0805_low_esl_cap_avx_w_via_dense
- removed R3: 10k, ftprnts:R_0201_0603Metric_dense
- removed SW1: SW_Push, ftprnts:EVPBL9A2B000
Connections:
- D2 pad 2: +3V3 -> LED2
- R2 pad 1: LED2 -> GND
- U1 pad A4: Net-(U1-PadA4) -> SWDCLK
- U1 pad B3: Net-(U1-PadB3) -> (no net)
- U1 pad B4: Net-(U1-PadB4) -> (no net)
- U1 pad B6: Net-(U1-PadB6) -> (no net)
- U1 pad B9: SWDCLK -> (no net)
- U1 pad C1: Net-(U1-PadC1) -> (no net)
- U1 pad C2: Net-(U1-PadC2) -> (no net)
- U1 pad C3: Net-(U1-PadC3) -> (no net)
- U1 pad C4: Net-(U1-PadC4) -> (no net)
- U1 pad C5: Net-(U1-PadC5) -> (no net)
- U1 pad C6: Net-(U1-PadC6) -> (no net)
- U1 pad C7: Net-(U1-PadC7) -> (no net)
- U1 pad D2: Net-(U1-PadD2) -> (no net)
- U1 pad D3: Net-(U1-PadD3) -> (no net)
- U1 pad D4: Net-(U1-PadD4) -> (no net)
- U1 pad D5: Net-(U1-PadD5) -> (no net)
- U1 pad D6: UART_TX -> (no net)
- U1 pad D7: Net-(U1-PadD7) -> (no net)
- U1 pad E1: Net-(U1-PadE1) -> (no net)
- U1 pad E4: Net-(U1-PadE4) -> (no net)
- U1 pad E6: Net-(U1-PadE6) -> (no net)
- U1 pad F1: Net-(U1-PadF1) -> (no net)
- U1 pad F2: Net-(U1-PadF2) -> (no net)
- U1 pad F3: Net-(U1-PadF3) -> (no net)
- U1 pad F4: Net-(U1-PadF4) -> (no net)
- U1 pad F6: Net-(U1-PadF6) -> (no net)
- U1 pad F8: XO -> (no net)
- U1 pad G2: Net-(U1-PadG2) -> (no net)
- U1 pad G3: Net-(U1-PadG3) -> (no net)
- U1 pad G4: Net-(U1-PadG4) -> (no net)
- U1 pad H1: Net-(U1-PadH1) -> (no net)
- U1 pad H2: Net-(U1-PadH2) -> (no net)
- U1 pad H3: Net-(U1-PadH3) -> (no net)
- U1 pad H4: Net-(U1-PadH4) -> (no net)
- U1 pad J2: Net-(U1-PadJ2) -> (no net)
- U1 pad J3: Net-(U1-PadJ3) -> (no net)
- U1 pad J8: Net-(U1-PadJ8) -> (no net)
Routing:
- net NRST: track 6.30 -> 0.08 mm, vias 2 -> 1
- net 3.3-5V_IN: track 6.67 -> 4.28 mm
- net +3V3: track 5.55 -> 4.51 mm
- net GND: track 4.50 -> 3.72 mm
- net Net-(D2-Pad1): track 0.68 -> 0.00 mm
- net LED2: track 6.53 -> 7.12 mm
